File: Hardware/Estação/Placa Mãe/Dev_1.3/RiMon.kicad_sch (KiCad schematic)
At the start: 58 parts, among them J1 PWR, J10 IO, J11 PGM2, J2 SNS_PWR, J3 Pluv, J4 JBAT, J5 Radio, J6 I2C, J7 LCD, J8 USS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

Commit message: Atualiza para Kicad 9.0
Other:
- note added: "2024-11-25"
- note added: "Dev 1.3"
- note added: "Estação de Monitoramento - Placa Mãe"
- note removed: "2024-05-22"
- note removed: "Dev 1.2"
- note removed: "Radio: LoRa RA-02"
- note removed: "Sensor de Chuva - Placa Mãe"
- note removed: "UART: CP2102N"
